Commit message: fixed rotating laserscan by changing the robot conf, make sure the origin of base link is at the center of both diff wheels, otherwise the offset will cause hundereds issues. now we have better accurate map

File: src/my_bot/urdf/my_robot.urdf (robot description, URDF)
Before this commit: robot my_robot, 5 links, 4 joints
Joints:
- joint caster_joint: origin xyz=0.2 0 -0.1 -> xyz=0.35 0 -0.1
- joint left_wheel_joint: origin xyz=-0.15 0.225 -0.05 rpy=-1.57 0 0 -> xyz=0 0.225 -0.05 rpy=-1.57 0 0
- joint right_wheel_joint: origin xyz=-0.15 -0.225 -0.05 rpy=-1.57 0 0 -> xyz=0 -0.225 -0.05 rpy=-1.57 0 0
