Commit message: simulation: reduce robot size, make it has a vaccum robot's size

File: src/simulation/urdf/my_robot.urdf (robot description, URDF)
Before this commit: robot my_robot, 5 links, 4 joints
Links:
- link base_link: mass 5.0 -> 1.0; geometry collision box size=0.3 0.2 0.1; visual box size=0.3 0.2 0.1
- link caster_wheel: mass 1.0 -> 2.0
- link left_wheel: geometry collision cylinder length=0.05 radius=0.05; visual cylinder length=0.05 radius=0.05
- link right_wheel: geometry collision cylinder length=0.05 radius=0.05; visual cylinder length=0.05 radius=0.05
Joints:
- joint caster_joint: origin xyz=0.35 0 -0.1 -> xyz=0.3 0 -0.05
- joint left_wheel_joint: origin xyz=0 0.225 -0.05 rpy=-1.57 0 0 -> xyz=0 0.125 -0.05 rpy=-1.57 0 0
- joint lidar_joint: origin xyz=0 0 0.12 rpy=0 0 0 -> xyz=0 0 0.07 rpy=0 0 0
- joint right_wheel_joint: origin xyz=0 -0.225 -0.05 rpy=-1.57 0 0 -> xyz=0 -0.125 -0.05 rpy=-1.57 0 0
